File: shift-triggers.sch (KiCad schematic (older format))
At the start: 32 parts, among them J1 output, P1 digiin, P2 digicascade, P3 MTA-156-4, P4 digiin-3v, U1 74HC595, U2 74HC595, U3 7805, U4 74LS125

Commit message: added ground, updated packages
Parts:
- added J2: gnd, Pin_Headers:Pin_Header_Straight_1x01_Pitch2.54mm, symbol Conn_01x01
- C1, C2: footprint Capacitors_THT:C_Disc_D4.3mm_W1.9mm_P5.00mm -> Capacitors_THT:C_Disc_D3.4mm_W2.1mm_P2.50mm
- C4, C5: footprint Capacitors_THT:C_Disc_D3.4mm_W2.1mm_P2.50mm -> Capacitors_THT:C_Disc_D4.3mm_W1.9mm_P5.00mm
Connections:
- net GND: now also J2.1 (Pin_1)
Changed lines of the file:
@@
 F 0 "C4" H 9425 1450 50  0000 L CNN
 F 1 "100n" H 9425 1250 50  0000 L CNN
-F 2 "Capacitors_THT:C_Disc_D3.4mm_W2.1mm_P2.50mm" H 9438 1200 50  0001 C CNN
+F 2 "Capacitors_THT:C_Disc_D4.3mm_W1.9mm_P5.00mm" H 9438 1200 50  0001 C CNN
 F 3 "" H 9400 1350 50  0000 C CNN
 	1    9400 1350
@@
 F 0 "C5" H 10325 1450 50  0000 L CNN
 F 1 "100n" H 10325 1250 50  0000 L CNN
-F 2 "Capacitors_THT:C_Disc_D3.4mm_W2.1mm_P2.50mm" H 10338 1200 50  0001 C CNN
+F 2 "Capacitors_THT:C_Disc_D4.3mm_W1.9mm_P5.00mm" H 10338 1200 50  0001 C CNN
 F 3 "" H 10300 1350 50  0000 C CNN
 	1    10300 1350
@@
 F 0 "C2" H 8325 3200 50  0000 L CNN
 F 1 "100n" H 8325 3000 50  0000 L CNN
-F 2 "Capacitors_THT:C_Disc_D4.3mm_W1.9mm_P5.00mm" H 8338 2950 50  0001 C CNN
+F 2 "Capacitors_THT:C_Disc_D3.4mm_W2.1mm_P2.50mm" H 8338 2950 50  0001 C CNN
 F 3 "" H 8300 3100 50  0000 C CNN
 	1    8300 3100
@@
 F 0 "C1" H 8075 3200 50  0000 L CNN
 F 1 "100n" H 8075 3000 50  0000 L CNN
-F 2 "Capacitors_THT:C_Disc_D4.3mm_W1.9mm_P5.00mm" H 8088 2950 50  0001 C CNN
+F 2 "Capacitors_THT:C_Disc_D3.4mm_W2.1mm_P2.50mm" H 8088 2950 50  0001 C CNN
 F 3 "" H 8050 3100 50  0000 C CNN
 	1    8050 3100
@@
 	10225 1550 10225 1700
 Connection ~ 10225 1550
+$Comp
+L Conn_01x01 J2
+U 1 1 5C1E6566
+P 6975 1275
+F 0 "J2" H 6975 1375 50  0000 C CNN
+F 1 "gnd" H 6975 1175 50  0000 C CNN
+F 2 "Pin_Headers:Pin_Header_Straight_1x01_Pitch2.54mm" H 6975 1275 50  0001 C CNN
+F 3 "" H 6975 1275 50  0001 C CNN
+	1    6975 1275
+	0    -1   -1   0
+$EndComp
+$Comp
+L GND #PWR012
+U 1 1 5C1E67D2
+P 6975 1575
+F 0 "#PWR012" H 6975 1325 50  0001 C CNN
+F 1 "GND" H 6975 1425 50  0000 C CNN
+F 2 "" H 6975 1575 50  0000 C CNN
+F 3 "" H 6975 1575 50  0000 C CNN
+	1    6975 1575
+	1    0    0    -1
+$EndComp
+Wire Wire Line
+	6975 1475 6975 1575
 $EndSCHEMATC

Commit message: mostly layed out now
Connections:
- net CLK: now also P1.3 (P3), P2.3 (P3); no longer P1.2 (P2), P2.2 (P2)
- net CLK-3v: now also P4.3 (P3); no longer P4.2 (P2)
- net CLR: now also P1.2 (P2), P2.2 (P2); no longer P1.3 (P3), P2.3 (P3)
- net CLR-3v: now also P4.2 (P2); no longer P4.3 (P3)
Changed lines of the file:
@@
 CLK
 Text GLabel 4925 1150 3    60   Input ~ 0
-CLK
+CLR
 Text GLabel 1050 1475 0    60   Output ~ 0
 CLR
@@
 RCLK
 Text GLabel 4775 1150 3    60   Input ~ 0
-CLR
+CLK
 Text GLabel 4625 1150 3    60   Input ~ 0
 RCLK
@@
 INSER-3v
 Text GLabel 4625 1800 2    60   Input ~ 0
+CLR-3v
+Text GLabel 4625 1925 2    60   Input ~ 0
 CLK-3v
-Text GLabel 4625 1925 2    60   Input ~ 0
-CLR-3v
 Text GLabel 4625 2050 2    60   Input ~ 0
 RCLK-3v
