File: shift-triggers.kicad_pcb (KiCad board)
At the start: 2 copper layers, 32 parts, among them J1 output, P1 digiin, P2 digicascade, P3 MTA-156-4, P4 digiin-3v, U1 74HC595, U2 74HC595, U3 7805, U4 74LS125

Commit message: more dialed in layout
Parts:
- added J2: gnd, Pin_Headers:Pin_Header_Straight_1x01_Pitch2.54mm, F.Cu at (108.6, 82.5)
- C1, C2: footprint Capacitors_THT:C_Disc_D4.3mm_W1.9mm_P5.00mm -> Capacitors_THT:C_Disc_D3.4mm_W2.1mm_P2.50mm
- C4, C5: footprint Capacitors_THT:C_Disc_D3.4mm_W2.1mm_P2.50mm -> Capacitors_THT:C_Disc_D4.3mm_W1.9mm_P5.00mm
- moved C4 36.5 mm to (104.9, 121.9), turned to 0 degrees
- moved C3 35.0 mm to (99.1, 121.3), turned to 90 degrees
- moved C1 31.0 mm to (95.9, 108.0), turned to 90 degrees
- moved C2 27.2 mm to (109.9, 88.9), turned to 90 degrees
- moved U3 27.2 mm to (98.4, 112.4), turned to 0 degrees
- moved U4 11.4 mm to (99.1, 86.4)
- moved R17 11.1 mm to (109.2, 126.4), turned to 180 degrees
- moved C6 11.0 mm to (95.9, 86.4), turned to 90 degrees
- moved U1 9.09 mm to (85.1, 105.4)
- moved U2 9.09 mm to (85.1, 83.8)
- moved P1 5.47 mm to (92.7, 78.7), turned to 270 degrees
- moved C5 5.13 mm to (99.1, 106.7)
- moved P3 5.01 mm to (111.1, 117.9), turned to 180 degrees
- moved P4 4.93 mm to (106.0, 78.7), turned to 270 degrees
- moved R4 2.95 mm to (72.4, 90.3)
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
Commit message: mostly layed out now
Parts:
- added REF**: srh, xnorman:wire-strain-relief-hole, F.Cu at (65.4, 82.5)
- added REF**: srh, xnorman:wire-strain-relief-hole, F.Cu at (65.4, 105.4)
- added REF**: srh, xnorman:wire-strain-relief-hole, F.Cu at (65.4, 108.0)
- added REF**: srh, xnorman:wire-strain-relief-hole, F.Cu at (65.4, 110.5)
- added REF**: srh, xnorman:wire-strain-relief-hole, F.Cu at (65.4, 113.0)
- added REF**: srh, xnorman:wire-strain-relief-hole, F.Cu at (65.4, 115.6)
- added REF**: srh, xnorman:wire-strain-relief-hole, F.Cu at (65.4, 118.1)
- added REF**: srh, xnorman:wire-strain-relief-hole, F.Cu at (65.4, 120.7)
- added REF**: srh, xnorman:wire-strain-relief-hole, F.Cu at (65.4, 85.1)
- added REF**: srh, xnorman:wire-strain-relief-hole, F.Cu at (65.4, 87.6)
- added REF**: srh, xnorman:wire-strain-relief-hole, F.Cu at (65.4, 90.2)
- added REF**: srh, xnorman:wire-strain-relief-hole, F.Cu at (65.4, 92.7)
- added REF**: srh, xnorman:wire-strain-relief-hole, F.Cu at (65.4, 95.2)
- added REF**: srh, xnorman:wire-strain-relief-hole, F.Cu at (65.4, 97.8)
- added REF**: srh, xnorman:wire-strain-relief-hole, F.Cu at (65.4, 100.3)
- added REF**: srh, xnorman:wire-strain-relief-hole, F.Cu at (65.4, 102.9)
- added REF1: MountingHole_3.2mm_M3, Mounting_Holes:MountingHole_3.2mm_M3, F.Cu at (67.9, 76.2)
- added REF2: MountingHole_3.2mm_M3, Mounting_Holes:MountingHole_3.2mm_M3, F.Cu at (112.4, 76.2)
- added REF3: MountingHole_3.2mm_M3, Mounting_Holes:MountingHole_3.2mm_M3, F.Cu at (112.4, 127.0)
- added REF4: MountingHole_3.2mm_M3, Mounting_Holes:MountingHole_3.2mm_M3, F.Cu at (67.9, 127.0)
- moved GND 2.54 mm to (111.1, 82.5)
- moved R17 1.91 mm to (107.3, 126.4)
- renumbered J2 to GND, P4 to IN-3v, P1 to IN-5v
Connections:
- IN-3v pad 2: CLK-3v -> CLR-3v
- IN-3v pad 3: CLR-3v -> CLK-3v
- IN-5v pad 2: CLK -> CLR
- IN-5v pad 3: CLR -> CLK
- P2 pad 2: CLK -> CLR
- P2 pad 3: CLR -> CLK
Routing:
- net RCLK: track 0.00 -> 75.4 mm, vias 0 -> 2
- net CLR: track 0.00 -> 69.6 mm
- net CLK: track 0.00 -> 64.3 mm, vias 0 -> 2
- net 5v: track 0.00 -> 62.2 mm
- net CLR-3v: track 0.00 -> 23.7 mm, vias 0 -> 1
- net Net-(C3-Pad1): track 0.00 -> 23.6 mm
- net CLK-3v: track 0.00 -> 20.7 mm
- net INSER: track 0.00 -> 19.2 mm
- net RCLK-3v: track 0.00 -> 19.1 mm, vias 0 -> 1
- net INSER-3v: track 0.00 -> 16.0 mm, vias 0 -> 1
- net trig8: track 0.00 -> 14.9 mm
- net trig0: track 0.00 -> 14.7 mm
- net Net-(P3-Pad1): track 0.00 -> 10.8 mm
- net trig4: track 0.00 -> 5.66 mm
- net trig1: track 0.00 -> 5.66 mm
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Other:
- net class Default: clearance 0.2 -> 0.1524; trace_width 0.25 -> 0.1524; via_dia 0.6 -> 0.6858; via_drill 0.4 -> 0.3302
- rule trace_clearance: 0.2 -> 0.1524
- rule trace_min: 0.2 -> 0.1524
- rule via_min_drill: 0.3 -> 0.3302
- rule via_min_size: 0.4 -> 0.6858
- board text added: "+"
- board text added: "1k"
- board text added: "rclk, clk, clr, inser"

Commit message: finalized pcb?
Routing:
- net Net-(U1-Pad14): track 0.00 -> 10.6 mm
- net GND: track 0.00 -> 3.19 mm
- net CLK: track 64.3 -> 65.6 mm
- net RCLK: track 75.4 -> 76.2 mm
- added copper zone on B.Cu, net GND
- added copper zone on F.Cu, net GND
Other:
- board outline added: 52.8 x 58.9 mm
- board text added: "by xnor dec-2018"
- board text added: "shift-trig"
Changed lines of the file:
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@@
 (kicad_pcb (version 4) (host pcbnew 4.0.7-e2-6376~60~ubuntu17.10.1)
   (general
-    (links 0)
-    (no_connects 39)
-    (area 0 0 0 0)
+    (links 81)
+    (no_connects 0)
+    (area 58.435457 71.0726 121.904543 132.2274)
     (thickness 1.6)
-    (drawings 3)
-    (tracks 145)
+    (drawings 9)
+    (tracks 160)
     (zones 0)
     (modules 53)
@@
     (47 F.CrtYd user)
     (48 B.Fab user)
-    (49 F.Fab user)
+    (49 F.Fab user hide)
   )
   (setup
@@
       (effects (font (size 1 1) (thickness 0.15)))
     )
-    (fp_text value 74HC595 (at 2.54 13.97 90) (layer F.SilkS)
+    (fp_text value 74HC595 (at 2.794 5.334 90) (layer F.SilkS)
       (effects (font (size 1 1) (thickness 0.15)))
     )
@@
       (effects (font (size 1 1) (thickness 0.15)))
     )
-    (fp_text value 74HC595 (at 2.54 13.97 90) (layer F.SilkS)
+    (fp_text value 74HC595 (at 2.794 5.08 90) (layer F.SilkS)
       (effects (font (size 1 1) (thickness 0.15)))
     )
@@
     (pad "" np_thru_hole circle (at 0 0) (size 2 2) (drill 1.9) (layers *.Cu *.Mask))
   )
+  (gr_text "by xnor\ndec-2018" (at 76.708 126.492) (layer F.SilkS)
+    (effects (font (size 1 1) (thickness 0.15)))
+  )
+  (gr_text shift-trig (at 113.792 93.472 90) (layer F.SilkS)
+    (effects (font (size 2 2) (thickness 0.3)))
+  )
+  (gr_line (start 116.332 131.064) (end 63.5 131.064) (layer Edge.Cuts) (width 0.15))
+  (gr_line (start 116.332 72.136) (end 116.332 131.064) (layer Edge.Cuts) (width 0.15))
+  (gr_line (start 63.5 72.136) (end 116.332 72.136) (layer Edge.Cuts) (width 0.15))
+  (gr_line (start 63.5 131.064) (end 63.5 72.136) (layer Edge.Cuts) (width 0.15))
   (gr_text + (at 112.395 120.65) (layer F.SilkS)
     (effects (font (size 1.5 1.5) (thickness 0.3)))
@@
     (effects (font (size 1.5 1.5) (thickness 0.3)))
   )
+  (segment (start 109.855 88.86) (end 106.72 88.86) (width 0.762) (layer F.Cu) (net 1))
+  (segment (start 106.72 88.86) (end 106.68 88.9) (width 0.762) (layer F.Cu) (net 1))
   (segment (start 111.188401 100.901599) (end 106.743401 105.346599) (width 0.762) (layer F.Cu) (net 2))
   (segment (start 100.473401 105.346599) (end 99.939999 105.880001) (width 0.762) (layer F.Cu) (net 2))
@@
   (segment (start 90.932 81.749) (end 92.71 79.971) (width 0.381) (layer B.Cu) (net 20))
   (segment (start 92.71 79.971) (end 92.71 78.74) (width 0.381) (layer B.Cu) (net 20))
+  (segment (start 88.9 96.012) (end 88.9 118.872) (width 0.381) (layer B.Cu) (net 21))
+  (segment (start 88.9 118.872) (end 88.9 125.73) (width 0.381) (layer B.Cu) (net 21))
+  (segment (start 88.9 118.11) (end 88.9 118.872) (width 0.381) (layer B.Cu) (net 21))
+  (segment (start 88.9 80.01) (end 88.9 96.012) (width 0.381) (layer B.Cu) (net 21))
+  (segment (start 88.9 96.52) (end 88.9 96.012) (width 0.381) (layer B.Cu) (net 21))
   (segment (start 99.06 99.06) (end 97.028 99.06) (width 0.381) (layer F.Cu) (net 21))
   (segment (start 97.028 99.06) (end 94.488 96.52) (width 0.381) (layer F.Cu) (net 21))
@@
   (via (at 88.9 96.52) (size 0.6858) (drill 0.3302) (layers F.Cu B.Cu) (net 21))
   (segment (start 87.63 78.74) (end 88.9 80.01) (width 0.381) (layer B.Cu) (net 21))
-  (segment (start 88.9 80.01) (end 88.9 125.73) (width 0.381) (layer B.Cu) (net 21))
   (segment (start 88.9 125.73) (end 87.63 127) (width 0.381) (layer B.Cu) (net 21))
   (segment (start 103.575 103.124) (end 97.174 103.124) (width 0.381) (layer F.Cu) (net 22))
@@
   (segment (start 90.17 99.06) (end 90.17 78.74) (width 0.381) (layer B.Cu) (net 22))
   (segment (start 92.71 99.06) (end 90.17 99.06) (width 0.381) (layer B.Cu) (net 22))
+  (segment (start 87.63 93.472) (end 87.63 115.824) (width 0.381) (layer B.Cu) (net 23))
+  (segment (start 87.63 115.824) (end 87.63 124.46) (width 0.381) (layer B.Cu) (net 23))
+  (segment (start 87.63 115.57) (end 87.63 115.824) (width 0.381) (layer B.Cu) (net 23))
+  (segment (start 87.63 82.482081) (end 87.63 93.472) (width 0.381) (layer B.Cu) (net 23))
+  (segment (start 87.63 93.98) (end 87.63 93.472) (width 0.381) (layer B.Cu) (net 23))
   (segment (start 106.68 93.98) (end 105.099 93.98) (width 0.381) (layer F.Cu) (net 23))
   (segment (start 105.099 93.98) (end 103.95609 95.12291) (width 0.381) (layer F.Cu) (net 23))
@@
   (segment (start 85.09 78.74) (end 85.09 79.942081) (width 0.381) (layer B.Cu) (net 23))
   (segment (start 85.09 79.942081) (end 87.63 82.482081) (width 0.381) (layer B.Cu) (net 23))
-  (segment (start 87.63 82.482081) (end 87.63 124.46) (width 0.381) (layer B.Cu) (net 23))
   (segment (start 87.63 124.46) (end 85.939999 126.150001) (width 0.381) (layer B.Cu) (net 23))
   (segment (start 85.939999 126.150001) (end 85.09 127) (width 0.381) (layer B.Cu) (net 23))
@@
   (segment (start 80.01 118.11) (end 85.09 118.11) (width 0.381) (layer F.Cu) (net 45))
   (segment (start 85.09 120.65) (end 80.01 120.65) (width 0.381) (layer F.Cu) (net 46))
+  (segment (start 90.932 104.559) (end 90.932 109.112) (width 0.381) (layer B.Cu) (net 47))
+  (segment (start 90.932 109.112) (end 92.31 110.49) (width 0.381) (layer B.Cu) (net 47))
+  (segment (start 92.31 110.49) (end 92.71 110.49) (width 0.381) (layer B.Cu) (net 47))
+  (segment (start 92.71 101.6) (end 92.71 102.781) (width 0.381) (layer B.Cu) (net 47))
+  (segment (start 92.71 102.781) (end 90.932 104.559) (width 0.381) (layer B.Cu) (net 47))
+  (zone (net 1) (net_name GND) (layer B.Cu) (hatch edge 0.508)
+    (connect_pads (clearance 0.508))
+    (min_thickness 0.254)
+    (fill yes (arc_segments 16) (thermal_gap 0.508) (thermal_bridge_width 0.508))
+    (polygon
+      (pts
+        (xy 115.824 72.644) (xy 64.008 72.644) (xy 64.008 130.556) (xy 115.824 130.556)
+      )
+    )
+  )
+  (zone (net 1) (net_name GND) (layer F.Cu) (hatch edge 0.508)
+    (connect_pads (clearance 0.508))
+    (min_thickness 0.254)
+    (fill yes (arc_segments 16) (thermal_gap 0.508) (thermal_bridge_width 0.508))
+    (polygon
+      (pts
+        (xy 115.824 72.644) (xy 64.008 72.644) (xy 64.008 130.556) (xy 115.824 130.556)
+      )
+    )
+  )
 )
